File: kicad/prototipo-stm32-nrf24l01/prototipo_gaspetto_car_bluepill.kicad_sch (KiCad schematic)
At the start: 19 parts, among them J1 Conn_01x07_Pin - TEST POINT, J2 NRF24L01_connector, J3 2x L911S connector, J4 Screw_Terminal_01x20, J5 Screw_Terminal_01x20, J6 Conn_01x04_Pin, M1 Motor_DC Right, M2 Motor_DC, Q1 BC548, U2 nRF24L01+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

Commit message: sch: create blackpill schematic
Parts:
- removed μC1, μC2: BlackPill, symbol muControllers_other:BlackPill
- added U1: YAAJ_BluePill_Part_Like_SWD_Breakout, symbol YAAJ_BluePill_Part_Like_SWD_Breakout:YAAJ_BluePill_Part_Like_SWD_Breakout
Connections:
- net 3v3: now also U3.6 (IA), U1.3 (PB14), U1.38 (3V3); no longer BZ1.1 (+), Q1.1 (C)
- net GND: now also U1.19 (GND), U1.39 (GND)
- net TX uC: now also U1.6 (PA9)
- net at U3.7 (IB): now also U1.4 (PB15)
- net at U6.23 (SCL): now also U1.14 (PB6)
- net at U6.24 (SDA): now also U1.15 (PB7)
- net at Q1.2 (B): now also U1.5 (PA8)
- net at U2.3 (CE): now also U1.27 (PA2)
- net at U2.4 (CSN): now also U1.29 (PA4)
- net at U2.5 (SCK): now also U1.30 (PA5)
- net at U2.6 (MOSI): now also U1.32 (PA7)
- net at U2.7 (MISO): now also U1.31 (PA6)
- net at U4.6 (IA): now also U1.36 (PB11)
- net at U4.7 (IB): now also U1.35 (PB10)
- new net: BZ1.1 (+), Q1.1 (C), U1.44 (3V3)
- no-connect marks 2 -> 0
Other:
- note added: "PA1 blackpill"
- note added: "PA3 blackpill"
- note added: "TIM1_CH2N"
- note added: "TIM1_CH3N"
- note added: "TIM2_CH3N"
- note added: "TIM2_CH4N"
- note added: "csn"
- note removed: "ALT RX uC"
- note removed: "ALT TX uC"
- note removed: "Buzzer - T4_CH4 (16 bit counter for PWM)"
- note removed: "CSN"
- note removed: "MISO"
- note removed: "MOSI"
- note removed: "SCK"
- note removed: "SCL1 I2C MPU"
- note removed: "SDA1 I2C MPU"
- note removed: "T2_CH1"
- note removed: "T2_CH2"
- note removed: "T2_CH3"
- note removed: "T2_CH4"
- note removed: "ok"
- note removed: "~RX uC 1~"
- note removed: "~TX uC 1~"
- moved on the sheet: U3
