File: kicad/prototipo-stm32-nrf24l01/prototipo_gaspetto_box.kicad_sch (KiCad schematic)
At the start: 19 parts, among them U1 YAAJ_BluePill_Part_Like_SWD_B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, U10 DRV5033AJxLPG, U11 DRV5033AJxLPG, U12 DRV5033AJxLPG, U13 DRV5033AJxLPG, U14 DRV5033AJxLPG, U15 DRV5033AJxLPG, U16 DRV5033AJxLPG, U17 DRV5033AJxLPG, U18 DRV5033AJxLPG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

Commit message: sch: work on Gaspetto Box schematics
Parts:
- removed U10, U11, U12, U13, U14, U15, U16, U17, U18, U19, U4, U5, U6, U7, U8, U9: DRV5033AJxLPG, Package_TO_SOT_THT:TO-92_Inline, symbol Sensor_Magnetic:DRV5033AJxLPG
- removed U3: PCF8575DBR, Package_SO:SSOP-24_5.3x8.2mm_P0.65mm, symbol Interface_Expansion:PCF8575DBR
- added U10, U11, U12, U13, U14, U15, U16, U17, U18, U19, U20, U21, U22, U23, U8, U9: DRV5055A1xLPGxQ1, Package_TO_SOT_THT:TO-92_Inline, symbol Sensor_Magnetic:DRV5055A1xLPGxQ1
- added U3, U4, U5, U6, U7: 74HC4051, symbol 74xx:74HC4051
- added μC1: BlackPill, symbol muControllers_other:BlackPill
Connections:
- new net: U3.3 (A), μC1.B1
- new net: U6.3 (A), μC1.A6
- new net: U5.3 (A), μC1.A7
- new net: U4.3 (A), μC1.B0
- new net: U7.3 (A), μC1.A5
Other:
- moved on the sheet: U1, U2
