File: kicad/prototipo-stm32-nrf24l01/prototipo_gaspetto_box.kicad_sch (KiCad schematic)
At the start: 60 parts, among them J1 UPS IN, J2 Conn_02x05_Odd_Even, J3 UPS OUT, J4 Conn_01x11, J5 Conn_02x05_Odd_Even, J6 Conn_02x05_Odd_Even, J7 Conn_01x11, P1 USB_C_Plug_USB2.0, Q1 AO3401A, Q2 AO3401A, U10 ADS1115IDGS, U11 DRV5033AJxLPG, U12 DRV5033AJxLPG, U13 DRV5033AJxLPG, U14 DRV5033AJxLPG, U15 ADS1115IDGS, U16 DRV5033AJxLPG, U17 DRV5033AJxLPG, U18 DRV5033AJxLPG, U19 DRV5033AJxLPG, U2 nRF24L01+, U20 ADS1115IDGS, U21 DRV5033AJxLPG, U22 DRV5033AJxLPG, U23 DRV5033AJxLPG, U24 DRV5033AJxLPG, U25 ADS1115IDGS, U26 DRV5033AJxLPG, U27 DRV5033AJxLPG, U28 DRV5033AJxLPG, U29 DRV5033AJxLPG, U3 MCP1700x-330xxTO, U30 MCP1700x-330xxTO, U31 YAAJ_WeAct_BlackPill_Part_Lik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, U4 ADS1115IDGS, U5 MCP1700x-330xxTO, U6 DRV5033AJxLPG, U7 DRV5033AJxLPG, U8 DRV5033AJxLPG, U9 DRV5033AJxLPG

Commit message: feat(gbox): add shared DFU bootloader entry and readable schematic
The DFU entry becomes a shared recipe: the production board and the
bench firmware jump to the bootloader the same way. The schematic is
reworked for readability and the scan header prints the EMPTY
threshold while dropping the unused LOOP_END.
Connections:
- net 3V3_SWITCHED: now also U15.1 (ADDR); no longer U25.1 (ADDR)
- net GND: no longer U20.1 (ADDR)
- net I2C1_SCL: now also U25.1 (ADDR); no longer U15.1 (ADDR)
- net I2C3_SDA: now also U20.1 (ADDR)
