File: kicad/prototipo-stm32-nrf24l01/prototipo_gaspetto_car.kicad_sch (KiCad schematic)
At the start: 18 parts, among them J1 Conn_01x07_Pin - TEST POINT, J2 NRF24L01_connector, J3 2x L911S connector, J4 Screw_Terminal_01x20, J5 Screw_Terminal_01x20, J6 Conn_01x04_Pin, M1 Motor_DC Right, M2 Motor_DC, Q1 BC548, U1 YAAJ_BluePill_Part_Like_SWD_B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

Commit message: sch: add blackpill new connections
Parts:
- removed U1: YAAJ_BluePill_Part_Like_SWD_Breakout, symbol YAAJ_BluePill_Part_Like_SWD_Breakout:YAAJ_BluePill_Part_Like_SWD_Breakout
- added μC1, μC2: BlackPill, symbol muControllers_other:BlackPill
Connections:
- net 3v3: now also BZ1.1 (+), Q1.1 (C), μC2.3.3ii; no longer U3.6 (IA)
- net RX uC: now also μC2.A10
- net TX uC: now also μC2.A9
- net at U6.23 (SCL): now also μC2.B6
- net at U6.24 (SDA): now also μC2.B7
- net at U2.3 (CE): now also μC2.B0
- net at U2.4 (CSN): now also μC2.B1
- net at U2.5 (SCK): now also μC2.A5
- net at U2.7 (MISO): now also μC2.A6
- net at U2.6 (MOSI): now also μC2.A7
- net at U4.7 (IB): now also μC2.A1
- net at U4.6 (IA): now also μC2.A0
- net at U3.7 (IB): now also μC2.A2
- net at Q1.2 (B): now also μC2.B9
- net SpeedSensor1 PA1: no longer names the net of J1.2 (Pin_2)
- net SpeedSensor2 PA0: no longer names the net of J1.5 (Pin_5)
- new net: U3.6 (IA), μC2.A3
- no-connect marks 1 -> 2
Other:
- note added: "ALT RX uC"
- note added: "ALT TX uC"
- note added: "Buzzer - T4_CH4 (16 bit counter for PWM)"
- note added: "CE"
- note added: "CSN"
- note added: "MISO"
- note added: "MOSI"
- note added: "SCK"
- note added: "SCL1 I2C MPU"
- note added: "SDA1 I2C MPU"
- note added: "T2_CH1"
- note added: "T2_CH2"
- note added: "T2_CH3"
- note added: "T2_CH4"
- note added: "ok"
- note added: "~RX uC 1~"
- note added: "~TX uC 1~"
- note removed: "TIM1_CH2N"
- note removed: "TIM1_CH3N"
- note removed: "TIM2_CH3N"
- note removed: "TIM2_CH4N"
- moved on the sheet: J1, J2, J3, J4, J5, U3
